File: pcb/main pcb/endev_v1.1.kicad_pcb (KiCad board)
At the start: 2 copper layers, 97.9 x 84.8 mm, 63 parts, among them J1 ICSP, J2 USB_C_Receptacle_USB2.0_16P, J3 Conn_01x03, J5 Conn_01x03, Q1 AO3401A, SW1 TS-1187A-B-A-B, SW2 JS102011JCQN, SW4 SW_DIP_x02, U1 ATmega328P-A, U10 SHT31-DIS, U2 CH340N, U3 LIS3DH, U5 TP4057, U6 XC6206P332MR, U7 ESP-12F, U8 ADG884xCP, Y1 16 MHz C13738

Commit message: fixed pcb
Parts:
- C15: footprint Capacitor_SMD:C_0805_2012Metric -> Capacitor_SMD:C_0402_1005Metric
- D27, D29: footprint LED_SMD:LED_0805_2012Metric -> LED_SMD:LED_0603_1608Metric
- J1: footprint Connector_PinSocket_2.00mm:PinSocket_2x03_P2.00mm_Vertical_SMD -> Connector_PinSocket_2.00mm:PinSocket_2x03_P2.00mm_Vertical
- J5: footprint Connector_PinHeader_2.54mm:PinHeader_1x03_P2.54mm_Vertical -> Connector_JST:JST_PH_B3B-PH-K_1x03_P2.00mm_Vertical
- U7: footprint endev_v1.1:ESP-12F -> RF_Module:ESP-12E
- moved R18 5.81 mm to (138.2, 114.5)
- moved J1 2.49 mm to (166.2, 104.2), turned to 0 degrees
- moved U7 2.20 mm to (151.9, 56.2)
- moved C16 1.83 mm to (140.8, 66.3)
- moved C15 1.81 mm to (142.0, 66.2)
- moved R15 1.70 mm to (161.8, 65.8)
- moved C17 1.20 mm to (140.2, 62.8)
- moved R17 1.14 mm to (145.2, 70.5), turned to 90 degrees
- moved R11 1.06 mm to (159.8, 70.2)
- moved D28 0.51 mm to (138.2, 112.0)
- moved Q1 0.45 mm to (136.6, 108.2)
- moved D25 0.09 mm to (140.8, 97.2)
- turned J5 to 90 degrees
- turned SW1 to 0 degrees
Routing:
- net /RESET: track 80.5 -> 89.0 mm, vias 7 -> 5
- net VCC: track 222.8 -> 229.3 mm, vias 15 -> 13
- net +BATT: track 25.4 -> 29.7 mm
- net D13: track 23.1 -> 27.3 mm
- net ESP_RXD: track 29.0 -> 32.4 mm
- net Net-(U7-~{RST}): track 1.74 -> 4.41 mm
- net D11: track 29.8 -> 27.7 mm
- net GND: track 86.1 -> 87.7 mm, vias 34 -> 31
- net D2: track 36.2 -> 37.3 mm
- net Net-(U7-GPIO0): track 11.4 -> 12.4 mm
- net Vdrive: track 45.9 -> 46.9 mm
- net Net-(U7-GPIO15): track 1.78 -> 2.45 mm
- net ESP_TXD: track 31.2 -> 31.9 mm, vias 0 -> 2
- net unconnected-(U7-GPIO5-Pad20): track 0.00 -> 0.60 mm
- net Net-(U7-EN): track 15.3 -> 15.8 mm, vias 2 -> 0
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Other:
- board size 97.9 x 84.8 mm -> 36 x 70 mm
