File: pcb/main pcb/endev_v1.1.kicad_sch (KiCad schematic)
At the start: 30 parts, among them J1 ICSP, J2 USB_C_Receptacle_USB2.0_16P, J5 Conn_01x03, SW1 TS-1187A-B-A-B, U1 ATmega328P-A, U2 CH340N, U7 ESP-12F, U8 ADG884xCP, Y1 16 MHz C13738

Commit message: fixed pcb
Parts:
- C1, C2: LCSC C14663 -> (none)
- C15: footprint Capacitor_SMD:C_0805_2012Metric -> Capacitor_SMD:C_0402_1005Metric; LCSC C15850 -> (none)
- C16, C5, C6, C7: LCSC C1525 -> (none)
- C3, C4: LCSC C1547 -> (none)
- D27: footprint LED_SMD:LED_0805_2012Metric -> LED_SMD:LED_0603_1608Metric; LCSC C2296 -> (none)
- D29: footprint LED_SMD:LED_0805_2012Metric -> LED_SMD:LED_0603_1608Metric; LCSC C2297 -> (none)
- D30: LCSC C8678 -> (none)
- J1: footprint Connector_PinSocket_2.00mm:PinSocket_2x03_P2.00mm_Vertical_SMD -> Connector_PinSocket_2.00mm:PinSocket_2x03_P2.00mm_Vertical
- J2: LCSC C2988369 -> (none)
- J5: footprint Connector_PinHeader_2.54mm:PinHeader_1x03_P2.54mm_Vertical -> Connector_JST:JST_PH_B3B-PH-K_1x03_P2.00mm_Vertical
- R1, R11, R15, R16, R17: LCSC C25744 -> (none)
- R13: LCSC C23138 -> (none)
- R2, R3: LCSC C25905 -> (none)
- SW1: LCSC C318884 -> (none)
- U1: LCSC C14877 -> (none)
- U2: LCSC C2977777 -> (none)
- U7: footprint endev_v1.1:ESP-12F -> RF_Module:ESP-12E; LCSC C82891 -> (none)
- U8: LCSC C140435 -> (none)
- Y1: LCSC C13738 -> (none)
